File: PCB/stm32_player/stm32_player.kicad_sch (KiCad schematic)
At the start: 8 parts, among them J1 ST1W008S4ER1500, U1 STM32L496ZGT6, U2 PCM5102A

Commit message: PCB to the cloud
Parts:
- added C10, C17, C18, C19, C9: 100nF, Capacitor_SMD:C_0402_1005Metric, symbol Device:C_Small
- added C11, C12, C23, C24, C26: 12pF, Capacitor_SMD:C_0402_1005Metric, symbol Device:C_Small
- added C13, C14, C22, C25: 820pF, Capacitor_SMD:C_0402_1005Metric, symbol Device:C_Small
- added C15, C16, C21, C27, C29, C30, C8: 4.7uF, Capacitor_SMD:C_0402_1005Metric, symbol Device:C_Small
- added C20, C6: 1uF, Capacitor_SMD:C_0402_1005Metric, symbol Device:C_Small
- added C28: 10uF, Capacitor_SMD:C_0402_1005Metric, symbol Device:C_Small
- added C31, C32, C33, C34, C35, C38, C39: 2.2, symbol Device:C_Small
- added C36, C37, C42, C43, C44, C45: 0.1, symbol Device:C_Small
- added C40, C41: 1uF, symbol Device:C_Small
- added C7: 47nF, Capacitor_SMD:C_0402_1005Metric, symbol Device:C_Small
- added D1: 1N4148, Diode_THT:D_DO-35_SOD27_P7.62mm_Horizontal, symbol Diode:1N4148
- added D5, D6, D63: LED, LED_SMD:LED_0402_1005Metric, symbol Device:LED
- added D62: ORANGE, LED_SMD:LED_0402_1005Metric, symbol Device:LED
- added J2: Battery Connector, Jumper:SolderJumper-2_P1.3mm_Bridged2Bar_Pad1.0x1.5mm, symbol Connector:Conn_01x02_Pin
- added J3: USB_C_Receptacle_USB2.0_16P, 12401598E4_2A:AMPHENOL_12401598E4_2A, symbol Connector:USB_C_Receptacle_USB2.0_16P
- added J4: 54-00174, 54-00174:TENSILITY_54-00174, symbol 54-00174:54-00174
- added J5: Conn_01x30_MountingPin, symbol Connector_Generic_MountingPin:Conn_01x30_MountingPin
- added JP1: Jumper_2_Bridged, Jumper:SolderJumper-2_P1.3mm_Bridged2Bar_Pad1.0x1.5mm, symbol Jumper:Jumper_2_Bridged
- added L1, L2, L4: 10uH, Inductor_SMD:L_0402_1005Metric, symbol Device:L
- added L3: 15nH, Inductor_SMD:L_0402_1005Metric, symbol Device:L
- added R1, R2: Resistor, Inductor_SMD:L_0402_1005Metric, symbol ScottoKeebs:Placeholder_Resistor
- added R10, R11: 5.1k, Inductor_SMD:L_0402_1005Metric, symbol ScottoKeebs:Placeholder_Resistor
- added R12, R13: 470, Inductor_SMD:L_0402_1005Metric, symbol ScottoKeebs:Placeholder_Resistor
- added R14, R19, R22, R9: 1k, Inductor_SMD:L_0402_1005Metric, symbol ScottoKeebs:Placeholder_Resistor
- added R15, R16, R17, R18: 22, Inductor_SMD:L_0402_1005Metric, symbol ScottoKeebs:Placeholder_Resistor
- added R20, R21, R5, R6, R7: 10k, Inductor_SMD:L_0402_1005Metric, symbol ScottoKeebs:Placeholder_Resistor
- added R3: 0, Inductor_SMD:L_0402_1005Metric, symbol ScottoKeebs:Placeholder_Resistor
- added R4: 2k, Inductor_SMD:L_0402_1005Metric, symbol ScottoKeebs:Placeholder_Resistor
- added R8: 10M, Inductor_SMD:L_0402_1005Metric, symbol ScottoKeebs:Placeholder_Resistor
- added SW1: Reset, Button_Switch_SMD:Panasonic_EVQPUJ_EVQPUA, symbol Switch:SW_Push
- added U3: NRF52840-QIAA-R7, NRF52840_QIAA_R7:NORDIC_NRF52840-QIAA-R7-2, symbol NRF52840-QIAA-R7:NRF52840-QIAA-R7
- added U4: XC6220B331MR, Package_TO_SOT_SMD:SOT-23-5, symbol Regulator_Linear:XC6220B331MR
- added U5: BQ24075TRGTR, BQ24075TRGTR:QFN50P300X300X100-17N, symbol BQ24075TRGTR:BQ24075TRGTR
- added U6, U7: ME6211C33M5, Package_TO_SOT_SMD:SOT-23-5, symbol Regulator_Linear:ME6211C33M5
- added Y1: XRCGB32M000F1H83R0, XRCGB32M000F1H8:OSC_XRCGB32M000F1H83R0, symbol XRCGB32M000F1H83R0:XRCGB32M000F1H83R0
- added Y2: FC-12M_32.7680KA-A3, FC-12M:XTAL_FC-12M_32.7680KA-A3, symbol FC-12M_32.7680KA-A3:FC-12M_32.7680KA-A3
Connections:
- net GND: now also J1.GND1 (GND), J1.GND2 (GND__1), J1.GND3 (GND__2), J1.GND4 (GND__3), U2.10 (DEMP), U2.11 (FLT), U2.9 (AGND), C10.1, C11.2, C12.2, C13.1, C14.1, C15.2, C16.1, C17.1, C18.1, C19.1, C20.1, C21.2, C22.1, C23.2, C24.2, C25.1, C26.2, C27.2, C28.2, C29.2, C30.2, C32.2, C33.2, C34.2, C35.2, C36.2, C37.2, C38.2, C39.2, C42.2, C43.1, C44.1, C45.1, C6.1, C7.1, C8.1, C9.1, D5.1 (K), D6.1 (K), J2.1 (Pin_1), J3.A1 (GND), J3.A12 (GND), J3.B1 (GND), J3.B12 (GND), J5.1 (Pin_1), J5.10 (Pin_10), J5.12 (Pin_12), J5.13 (Pin_13), J5.15 (Pin_15), J5.16 (Pin_16), J5.17 (Pin_17), J5.21 (Pin_21), J5.22 (Pin_22), J5.23 (Pin_23), J5.24 (Pin_24), J5.25 (Pin_25), J5.30 (Pin_30), J5.8 (Pin_8), J5.MP (MountPin), R10.1, R11.1, R22.1, R4.2, R5.1, R6.1, R9.1, U3.B7 (VSS), U4.2 (GND), U5.15 (SYSOFF), U5.4 (~{CE}), U5.5 (EN2), U5.8 (VSS), U7.2 (V_{SS})
- net SDMMC1_CK: now also J1.5
- net SDMMC1_CMD: now also J1.3
- net SDMMC1_D0: now also J1.7
- net SDMMC1_D1: now also J1.8
- net SDMMC1_D2: now also J1.1
- net SDMMC1_D3: now also J1.2
- net at C3.2, C5.2: now also C38.1, C39.1, U7.5 (V_{OUT})
- net at U2.1 (CPVDD): now also U2.8 (AVDD), C34.1, C35.1, R14.2, U6.5 (V_{OUT})
- net at U2.12 (SCK): now also R18.1
- net at U2.13 (BCK): now also R17.1
- net at U2.14 (DIN): now also R16.1
- net at U2.15 (LRCK): now also R15.1
- net at U2.2 (CAPP): now also C31.1
- net at U2.4 (CAPM): now also C31.2
- net at U2.6 (OUTL): now also R12.2
- net at U2.7 (OUTR): now also R13.2
- net VDD: now reaches J1.4
- net VSS: now reaches J1.6
- new net: C8.2, U3.AC5 (DECUSB)
- new net: J3.B5 (CC2), R11.2
- new net: J5.26 (Pin_26), R22.2
- new net: C6.2, C7.2, L3.1, U3.B5 (DEC4), U3.E24 (DEC6)
- new net: C43.2, J5.27 (Pin_27)
- new net: D62.1 (K), U5.9 (~{CHG})
- new net: D62.2 (A), R7.2
- new net: C22.2, L4.2, R3.1
- new net: C11.1, U3.F2 (P0.01/XL2), Y2.1
- new net: JP1.1 (A), R5.2, U5.16 (ISET)
- new net: C42.1, D1.2 (A), J5.14 (Pin_14), R19.1
- new net: C40.1, J5.2 (Pin_2)
- new net: C44.2, J5.28 (Pin_28)
- new net: C45.2, J5.29 (Pin_29)
- new net: C40.2, J5.3 (Pin_3)
- new net: C41.1, J5.4 (Pin_4)
- new net: C41.2, J5.5 (Pin_5)
- new net: C12.1, U3.D2 (P0.00/XL1), Y2.2
- new net: C14.2, L4.1, U3.H23 (ANT)
- new net: C23.1, U3.B24 (XC1), Y1.1
- new net: L1.2, U3.AB2 (DCCH)
- new net: C24.1, U3.A23 (XC2), Y1.3
- new net: C32.1, R13.1
- new net: J2.2 (Pin_2), U3.G1 (P0.26)
- new net: C36.1, C37.1, U6.1 (V_{IN}), U6.3 (CE), U7.1 (V_{IN}), U7.3 (CE)
- new net: J3.A5 (CC1), R10.2
- new net: L2.2, U3.B3 (DCC)
- new net: C9.2, U3.C1 (DEC1)
- new net: C10.2, U3.D23 (DEC3)
- new net: C13.2, U3.N24 (DEC5)
- new net: D6.2 (A), R2.1
- new net: R2.2, U3.T23 (P1.05)
- new net: L2.1, L3.2
- new net: JP1.2 (B), R4.1
- new net: D63.1 (K), R9.2
- new net: SW1.1, U3.AC17 (P0.21)
- new net: SW1.2, U3.AD16 (P0.20)
- new net: D5.2 (A), R1.1
- new net: R1.2, U3.R24 (P1.06)
- new net: D1.1 (K), R19.2
- new net: R6.2, U5.1 (TS)
- new net: C33.1, R12.1
- new net ANTENNA: C25.2, R3.2
- new net BCK: R17.2
- new net BLED: U3.AD10 (P0.15)
- new net C1: U3.B19 (P1.11)
- new net C2: U3.B17 (P1.12)
- new net C3: U3.A16 (P1.13)
- new net C4: U3.B15 (P1.14)
- new net D+: J3.A6 (D+), J3.B6 (D+), U3.AD6 (D+)
- new net D-: J3.A7 (D-), J3.B7 (D-), U3.AD4 (D-)
- new net DIN: R16.2
- new net ENC_A: U3.P2 (P1.08)
- new net ENC_B: U3.R1 (P1.09)
- new net EXT_VCC: C29.1, U4.5 (VOUT)
- new net LRCK: R15.2
- new net POWER_PIN: R8.1, U3.AD8 (P0.13), U4.3 (CE)
- new net RESET: U3.AC11 (P0.16), U3.AC13 (P0.18/~{RESET}), U3.AC9 (P0.14)
- new net RXD: U3.N1 (P0.08)
- new net SCK: R18.2
- new net SCL: J5.18 (Pin_18), R20.2
- new net SDA: J5.19 (Pin_19), J5.20 (Pin_20), R21.1
- new net SWC: U3.AA24 (SWDCLK)
- new net SWD: U3.AC24 (SWDIO)
- new net TXD: U3.L1 (P0.06)
- new net VBAT: C27.1, U5.2 (BAT), U5.3 (BAT__1)
- new net VBUS: C15.1, C21.1, C26.1, D63.2 (A), J3.A4 (VBUS), J3.A9 (VBUS), J3.B4 (VBUS), J3.B9 (VBUS), U3.AD2 (VBUS), U3.Y2 (VDDH), U5.13 (IN)
- new net VCC: J5.11 (Pin_11), J5.6 (Pin_6), J5.9 (Pin_9), R20.1, R21.2
- new net VDDH: C28.1, C30.1, R7.1, R8.2, U4.1 (VIN), U5.10 (OUT), U5.11 (OUT__1), U5.6 (EN1)
- new net VDD_NRF: C16.2, C17.2, C18.2, C19.2, C20.2, L1.1, U3.A22 (VDD)
- new net VSS_PA: U3.F23 (VSS_PA)
- no-connect marks 0 -> 7
Other:
- note added: "Charging and Power Path"
- note added: "Status LED"
- note added: "USB Port"
- note added: "VCC Regulator and Cut Off"
- note removed: "Battery Management System"
- moved on the sheet: C1, C2, C3, C4, C5, J1, U2
